File: PCB/splitkb.kicad_pcb (KiCad board)
At the start: 2 copper layers, 273.9 x 100.5 mm, 98 parts, among them J1 JST_2mm_LiPo, J2 JST_2mm_LiPo, M1 Module_XIAO-ESP32C3, M2 Module_XIAO-ESP32C3, SW1 RotaryEncoder, SW2 RotaryEncoder

Commit message: modified pcb and production files
Parts:
- SW1, SW2: footprint Rotary_Encoder:RotaryEncoder_Alps_EC12E_Vertical_H20mm -> zLibrary:RotaryEncoder_Alps_EC12E-Switch_Vertical_H20mm
- moved H11 38.1 mm to (205.2, 67.5)
- moved H6 33.3 mm to (225.1, 67.5)
- moved H4 30.8 mm to (231.8, 98.5)
- moved H2 21.4 mm to (350.1, 38.0)
- moved H10 21.2 mm to (350.1, 91.0)
- moved H1 19.1 mm to (81.7, 39.5)
- moved H3 18.8 mm to (81.3, 89.8)
- moved H12 6.09 mm to (296.7, 33.9)
- moved H5 5.54 mm to (133.4, 34.2)
- moved H7 5.22 mm to (172.8, 39.1)
- moved H8 4.39 mm to (257.2, 39.5)
- moved H9 1.46 mm to (198.1, 98.4)
Routing:
- net /right/C5: track 219.6 -> 191.3 mm, vias 0 -> 1
Other:
- outline, holes or cut-outs redrawn
